File: hardware/io-16.kicad_pcb (KiCad board)
At the start: 2 copper layers, 75 x 35 mm, 32 parts, among them J1 AKL_5_2, J10 AKL_5_2, J11 AKL_5_2, J12 AKL_5_2, J13 AKL_5_2, J2 AKL_5_2, J3 AKL_5_2, J4 AKL_5_2, J5 AKL_5_2, J6 AKL_5_2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

Commit message: Add 3d information (final)
Parts:
- C1, C2, C3: footprint 0603E -> kicad-libraries:C0603E
- Fiducial_Mark (x2): footprint Fiducial_Mark -> kicad-libraries:Fiducial_Mark
- J1, J10, J11, J12, J13, J2, J3, J4, J5, J6, J7, J8, J9: footprint AKL_5_2 -> kicad-libraries:AKL_5_2
- P1: footprint CON-SENSOR -> kicad-libraries:CON-SENSOR
- R1: footprint 0603E -> kicad-libraries:R0603E
- Ref**: footprint Logo_31x31 -> kicad-libraries:Logo_31x31
- U1: footprint TSSOP8 -> kicad-libraries:TSSOP8
- U2: footprint SOIC28 -> kicad-libraries:SOIC28
- U3: footprint TSSOP8_3 -> kicad-libraries:TSSOP8_3
- VAL: footprint CE_5mm -> kicad-libraries:CE_5mm
- VAL: footprint WEEE_7mm -> kicad-libraries:WEEE_7mm
- turned VAL to 180 degrees
Connections:
- P1 pad 10: (no net) -> Net-(P1-Pad10)
- P1 pad 9: (no net) -> Net-(P1-Pad9)
- RP1 pad 6: (no net) -> Net-(RP1-Pad6)
- RP1 pad 7: (no net) -> Net-(RP1-Pad7)
- SW1 pad 4: (no net) -> Net-(SW1-Pad4)
- SW1 pad 5: (no net) -> Net-(SW1-Pad5)
- SW1 pad 6: (no net) -> Net-(SW1-Pad6)
- U1 pad 7: (no net) -> Net-(U1-Pad7)
- U2 pad 11: (no net) -> Net-(U2-Pad11)
- U2 pad 14: (no net) -> Net-(U2-Pad14)
